File: led-matrix.kicad_pcb (KiCad board)
At the start: 2 copper layers, 89 x 66 mm, 91 parts, among them U1 MAX7219, U2 Pico

Commit message: feat: prep for ordering and add jlc order mark
Other:
- board text added: "JLCJLCJLCJLC"
Changed lines of the file:
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@@
 		(layer "Edge.Cuts")
+	)
+	(gr_text "JLCJLCJLCJLC"
+		(at 100.5 86.5 0)
+		(layer "F.Cu")
+		(effects
+			(font
+				(size 0.8 0.8)
+				(thickness 0.125)
+			)
+			(justify left bottom)
+		)
 	)
 	(gr_text "@kcoderhtml @wanderer.archives"

Commit message: feat: add logos
Parts:
- added face: LOGO, LOGO, B.Cu at (105.5, 85.0)
Other:
- board text added: "WayWayWay"
- board text added: "a kieran klukas and a wanderer's archives project"
- board text added: "sponsered by pcbway and made for the love of making"
- board text removed: "@kcoderhtml @wanderer.archives"
- board text removed: "JLCJLCJLCJLC"
